File: kicad_projects/EC2025/EC2025.kicad_sch (KiCad schematic)
At the start: 11 parts

Commit message: regular
Parts:
- added D1: ${SIM.PARAMS}, symbol 1_EC2019:DIODE
- added R9: R_Small_US, symbol Device:R_Small_US
- 60V, I1: Spice_Netlist_Enabled Y -> (none)
Connections:
- net GND: now also D1.2 (K)
- new net: D1.1 (A), R9.2
- new net +5V: R9.1
