File: kicad_projects/260103-esp32_demo-techExp/ESP32-C3-02.kicad_sch (KiCad schematic)
At the start: 30 parts, among them J3 GSD090012SEU, U3 ESP32-C3-WROOM-02-H4, U4 CP2102N-Axx-xQFN20, U5 USBLC6-2SC6, U6 W25Q32JVSSIQ

Commit message: regular
Parts:
- C10, C11, C14, C8: footprint (none) -> Capacitor_SMD:C_0805_2012Metric
- C12: renamed from C13; footprint (none) -> esp32_demo_footprints:T491A
- C13: renamed from C12; footprint (none) -> Capacitor_SMD:C_0805_2012Metric
- C7, C9: footprint (none) -> esp32_demo_footprints:T491A
- J3: footprint GSD090012SEU:AMPHENOL_GSD090012SEU -> esp32_demo_footprints:AMPHENOL_GSD090012SEU
- LED5: renamed from LED6; footprint LEDC2012X120N -> esp32_demo_footprints:LEDC2012X120N
- LED6: renamed from LED5; footprint LEDC2012X120N -> esp32_demo_footprints:LEDC2012X120N
- R11, R12, R13, R15, R16, R19, R20, R22: footprint (none) -> Resistor_SMD:R_0805_2012Metric
- R14, R18: value 470 -> 330; footprint (none) -> Resistor_SMD:R_0805_2012Metric
- TP1, TP2, TP3, TP4, TP5: footprint (none) -> TestPoint:TestPoint_Pad_D1.0mm
- U3: footprint ESP32-C3-WROOM-02-H4:MODULE_ESP32-C3-WROOM-02-H4 -> esp32_demo_footprints:MODULE_ESP32-C3-WROOM-02-H4
- U6: footprint W25Q32JVSSIQ:SOIC127P790X216-8N -> esp32_demo_footprints:SOIC127P790X216-8N
Connections:
- net DTS renamed DTR
Other:
- sheet Sensors ports: added MIC_OUT, PHOTO_C, SCL, SDA; removed none
- sheet User_interface ports: added BOOT, DTR, EN, GPIO18, GPIO19, GPIO8, RTS, SCL, SDA; removed none

Commit message: regular
Parts:
- U4: footprint Package_DFN_QFN:SiliconLabs_QFN-20-1EP_3x3mm_P0.5mm -> Package_DFN_QFN:SiliconLabs_QFN-20-1EP_3x3mm_P0.5mm_EP1.8x1.8mm
Changed lines of the file:
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@@
 			)
 		)
-		(property "Footprint" "Package_DFN_QFN:SiliconLabs_QFN-20-1EP_3x3mm_P0.5mm"
+		(property "Footprint" "Package_DFN_QFN:SiliconLabs_QFN-20-1EP_3x3mm_P0.5mm_EP1.8x1.8mm"
 			(at 116.84 110.49 0)
 			(effects
