File: kicad_projects/260103-esp32_demo-techExp/User_interface.kicad_sch (KiCad schematic)
At the start: 0 parts

Commit message: regular
Parts:
- added C21: 100n, Capacitor_SMD:C_0805_2012Metric, symbol Device:C
- added C22: 1u, Capacitor_SMD:C_0805_2012Metric, symbol Device:C
- added J4: Conn_01x04_Pin, Connector_PinHeader_2.54mm:PinHeader_1x04_P2.54mm_Vertical, symbol Connector:Conn_01x04_Pin
- added J5: Conn_01x05_Pin, Connector_PinHeader_2.54mm:PinHeader_1x05_P2.54mm_Vertical, symbol Connector:Conn_01x05_Pin
- added Q2, Q3: BC817, Package_TO_SOT_SMD:SOT-23, symbol Transistor_BJT:BC817
- added R32, R33, R34: 10k, Resistor_SMD:R_0805_2012Metric, symbol Device:R
- added S1, S2: USLPT2819DT2TR, esp32_demo_footprints:SW_USLPT2819DT2TR, symbol USLPT2819DT2TR:USLPT2819DT2TR
Connections:
- new net: Q2.1 (B), R33.2
- new net: Q3.1 (B), R34.2
- new net +3.3V: J4.1 (Pin_1), J5.1 (Pin_1), R32.2
- new net BOOT: C21.1, Q3.3 (C), S1.3, S1.4
- new net DTR: Q3.2 (E), R33.1
- new net EN: C22.1, Q2.3 (C), R32.1, S2.3, S2.4
- new net GND: C21.2, C22.2, J4.4 (Pin_4), J5.5 (Pin_5), S1.1, S1.2, S2.1, S2.2
- new net GPIO18: J5.3 (Pin_3)
- new net GPIO19: J5.4 (Pin_4)
- new net GPIO8: J5.2 (Pin_2)
- new net RTS: Q2.2 (E), R34.1
- new net SCL: J4.3 (Pin_3)
- new net SDA: J4.2 (Pin_2)
Other:
- note added: "OLED connector (I2C)"
- note added: "RST and BOOT buttons"
- note added: "Remaining GPIO pins"
