File: kicad_projects/260103-esp32_demo-techExp/260103-esp32_demo-techExp.kicad_pcb (KiCad board)
At the start: 4 copper layers, 0 parts

Commit message: regular
Parts:
- added C1: 100n, Capacitor_SMD:C_0805_2012Metric, F.Cu at (187.0, 75.2)
- added C10: 100n, Capacitor_SMD:C_0805_2012Metric, F.Cu at (148.2, 89.6)
- added C11: 1u, Capacitor_SMD:C_0805_2012Metric, F.Cu at (148.2, 92.6)
- added C12: 10u, esp32_demo_footprints:T491A, F.Cu at (155.3, 68.0)
- added C13: 100n, Capacitor_SMD:C_0805_2012Metric, F.Cu at (148.2, 95.6)
- added C14: 100n, Capacitor_SMD:C_0805_2012Metric, F.Cu at (148.2, 98.6)
- added C15: 100n, Capacitor_SMD:C_0805_2012Metric, F.Cu at (166.3, 89.2)
- added C16: 100n, Capacitor_SMD:C_0805_2012Metric, F.Cu at (166.3, 92.2)
- added C18: 100n, Capacitor_SMD:C_0805_2012Metric, F.Cu at (166.3, 95.2)
- added C2: 100n, Capacitor_SMD:C_0805_2012Metric, F.Cu at (187.0, 78.2)
- added C20: 100n, Capacitor_SMD:C_0805_2012Metric, F.Cu at (166.3, 98.2)
- added C21: 100n, Capacitor_SMD:C_0805_2012Metric, F.Cu at (128.2, 122.3)
- added C22: 1u, Capacitor_SMD:C_0805_2012Metric, F.Cu at (128.2, 125.3)
- added C3: 10u, esp32_demo_footprints:T491A, F.Cu at (181.3, 76.0)
- added C4: 10u, esp32_demo_footprints:T491A, F.Cu at (181.3, 80.6)
- added C5: 100n, Capacitor_SMD:C_0805_2012Metric, F.Cu at (187.0, 81.2)
- added C6: 1u, Capacitor_SMD:C_0805_2012Metric, F.Cu at (187.0, 84.2)
- added C7: 10u, esp32_demo_footprints:T491A, F.Cu at (155.3, 58.7)
- added C8: 100n, Capacitor_SMD:C_0805_2012Metric, F.Cu at (148.2, 86.6)
- added C9: 4u7, esp32_demo_footprints:T491A, F.Cu at (155.3, 63.3)
- added F1: 0ZCH0110AF2E, esp32_demo_footprints:FUSC3226X100N, F.Cu at (190.5, 58.5)
- added FB1: FBMJ2125HM330-T, esp32_demo_footprints:BEADC2012X105N, F.Cu at (189.9, 62.2)
- added J1: SS-52400-002, esp32_demo_footprints:BELFUSE_SS-52400-002, F.Cu at (169.7, 65.4)
- added J2: B2B-PH-SM4-TB, esp32_demo_footprints:JST_B2B-PH-SM4-TB, F.Cu at (182.7, 59.6)
- added J3: GSD090012SEU, esp32_demo_footprints:AMPHENOL_GSD090012SEU, F.Cu at (99.8, 112.8)
- added J4: Conn_01x04_Pin, Connector_PinHeader_2.54mm:PinHeader_1x04_P2.54mm_Vertical, F.Cu at (128.3, 110.9)
- added J5: Conn_01x05_Pin, Connector_PinHeader_2.54mm:PinHeader_1x05_P2.54mm_Vertical, F.Cu at (123.7, 110.9)
- added LED1: LTST-C170KRKT, esp32_demo_footprints:LEDC2012X120N, F.Cu at (175.3, 72.3)
- added LED2: LTST-C170GKT, esp32_demo_footprints:LEDC2012X120N, F.Cu at (175.3, 75.6)
- added LED3: LTST-C170TBKT, esp32_demo_footprints:LEDC2012X120N, F.Cu at (175.3, 79.0)
- added LED4: LTST-C170KRKT, esp32_demo_footprints:LEDC2012X120N, F.Cu at (175.3, 82.3)
- added LED5: LTST-C170GKT, esp32_demo_footprints:LEDC2012X120N, F.Cu at (154.1, 78.9)
- added LED6: LTST-C170KRKT, esp32_demo_footprints:LEDC2012X120N, F.Cu at (154.1, 82.3)
- added MK1: CMC-5042PF-AC, esp32_demo_footprints:CUI_CMC-5042PF-AC, F.Cu at (172.3, 100.3)
- added Q1: TEMT6000X01, esp32_demo_footprints:TRANS_TEMT6000X01, F.Cu at (172.3, 106.0)
- added Q2: BC817, Package_TO_SOT_SMD:SOT-23, F.Cu at (133.0, 110.8)
- added Q3: BC817, Package_TO_SOT_SMD:SOT-23, F.Cu at (133.0, 115.3)
- added R1: 10k, Resistor_SMD:R_0805_2012Metric, F.Cu at (166.3, 72.1)
- added R10: 330, Resistor_SMD:R_0805_2012Metric, F.Cu at (170.7, 83.9)
- added R11: 1k, Resistor_SMD:R_0805_2012Metric, F.Cu at (152.6, 86.5)
- added R12: 22k1, Resistor_SMD:R_0805_2012Metric, F.Cu at (152.6, 89.5)
- added R13: 47k5, Resistor_SMD:R_0805_2012Metric, F.Cu at (152.6, 92.4)
- added R14: 330, Resistor_SMD:R_0805_2012Metric, F.Cu at (152.6, 95.4)
- added R15: 50, Resistor_SMD:R_0805_2012Metric, F.Cu at (152.6, 98.3)
- added R16: 50, Resistor_SMD:R_0805_2012Metric, F.Cu at (157.0, 86.5)
- added R18: 330, Resistor_SMD:R_0805_2012Metric, F.Cu at (157.0, 89.5)
- added R19: 10k, Resistor_SMD:R_0805_2012Metric, F.Cu at (157.0, 92.4)
- added R2: 10k, Resistor_SMD:R_0805_2012Metric, F.Cu at (166.3, 75.0)
- added R20: 50, Resistor_SMD:R_0805_2012Metric, F.Cu at (157.0, 95.4)
- added R22: 50, Resistor_SMD:R_0805_2012Metric, F.Cu at (157.0, 98.3)
- added R23: 10k, Resistor_SMD:R_0805_2012Metric, F.Cu at (170.8, 89.2)
- added R24: 4k7, Resistor_SMD:R_0805_2012Metric, F.Cu at (170.8, 92.1)
- added R25: 4k7, Resistor_SMD:R_0805_2012Metric, F.Cu at (170.8, 95.1)
- added R26: 2k, Resistor_SMD:R_0805_2012Metric, F.Cu at (175.2, 89.2)
- added R27: 1M, Resistor_SMD:R_0805_2012Metric, F.Cu at (175.2, 92.1)
- added R28: 2k, Resistor_SMD:R_0805_2012Metric, F.Cu at (175.2, 95.1)
- added R29: 1M, Resistor_SMD:R_0805_2012Metric, F.Cu at (179.6, 89.2)
- added R3: 5k1, Resistor_SMD:R_0805_2012Metric, F.Cu at (166.3, 78.0)
- added R30: 10k, Resistor_SMD:R_0805_2012Metric, F.Cu at (179.6, 92.1)
- added R31: 100k, Resistor_SMD:R_0805_2012Metric, F.Cu at (179.6, 95.1)
- added R32: 10k, Resistor_SMD:R_0805_2012Metric, F.Cu at (137.7, 110.1)
- added R33: 10k, Resistor_SMD:R_0805_2012Metric, F.Cu at (137.7, 113.0)
- added R34: 10k, Resistor_SMD:R_0805_2012Metric, F.Cu at (137.7, 116.0)
- added R4: 5k1, Resistor_SMD:R_0805_2012Metric, F.Cu at (166.3, 80.9)
- added R5: 2k, Resistor_SMD:R_0805_2012Metric, F.Cu at (166.3, 83.9)
- added R6: 20k, Resistor_SMD:R_0805_2012Metric, F.Cu at (170.7, 72.1)
- added R7: 470, Resistor_SMD:R_0805_2012Metric, F.Cu at (170.7, 75.0)
- added R8: 470, Resistor_SMD:R_0805_2012Metric, F.Cu at (170.7, 78.0)
- added R9: 470, Resistor_SMD:R_0805_2012Metric, F.Cu at (170.7, 80.9)
- added S1: USLPT2819DT2TR, esp32_demo_footprints:SW_USLPT2819DT2TR, F.Cu at (133.5, 119.2)
- added S2: USLPT2819DT2TR, esp32_demo_footprints:SW_USLPT2819DT2TR, F.Cu at (133.5, 122.7)
- added TP1: Test MOSI, TestPoint:TestPoint_Pad_D1.0mm, F.Cu at (144.4, 86.6)
- added TP2: Test MISO, TestPoint:TestPoint_Pad_D1.0mm, F.Cu at (144.4, 89.6)
- added TP3: Test SCLK, TestPoint:TestPoint_Pad_D1.0mm, F.Cu at (144.4, 92.7)
- added TP4: Test CS_SD, TestPoint:TestPoint_Pad_D1.0mm, F.Cu at (144.4, 95.7)
- added TP5: Test CS, TestPoint:TestPoint_Pad_D1.0mm, F.Cu at (144.4, 98.8)
- added U1: MCP73871-2CAI_ML, esp32_demo_footprints:QFN50P400X400X100-21N, F.Cu at (190.3, 69.1)
- added U2: LM1117MPX-3.3, esp32_demo_footprints:VREG_LM1117MPX-3.3, F.Cu at (182.2, 69.8)
- added U3: ESP32-C3-WROOM-02-H4, esp32_demo_footprints:MODULE_ESP32-C3-WROOM-02-H4, F.Cu at (106.2, 75.2)
- added U4: CP2102N-Axx-xQFN20, Package_DFN_QFN:SiliconLabs_QFN-20-1EP_3x3mm_P0.5mm_EP1.8x1.8mm, F.Cu at (224.8, 111.0)
- added U5: USBLC6-2SC6, Package_TO_SOT_SMD:SOT-23-6, F.Cu at (159.1, 79.6)
- added U6: W25Q32JVSSIQ, esp32_demo_footprints:SOIC127P790X216-8N, F.Cu at (156.9, 73.8)
- added U7: BME280, esp32_demo_footprints:PSON65P250X250X100-8N, F.Cu at (178.2, 98.6)
- added U8: MAX4466EXK, esp32_demo_footprints:SOT65P210X110-5N, F.Cu at (178.9, 102.6)
- added VR1: LM1117MPX-3.3, esp32_demo_footprints:VREG_LM1117MPX-3.3, F.Cu at (226.6, 102.5)

Commit message: regular
Parts:
- removed U2: LM1117MPX-3.3, esp32_demo_footprints:VREG_LM1117MPX-3.3
- added C17: 10n, Capacitor_SMD:C_0805_2012Metric, F.Cu at (90.8, 65.0)
- added C19: 1u, Capacitor_SMD:C_0805_2012Metric, F.Cu at (96.0, 60.3)
- added REF**: MountingHole_2.5mm_Pad_Via, MountingHole:MountingHole_2.5mm_Pad_Via, F.Cu at (131.9, 89.8)
- added REF**: MountingHole_2.5mm_Pad_Via, MountingHole:MountingHole_2.5mm_Pad_Via, F.Cu at (114.1, 53.2)
- added REF**: MountingHole_2.5mm_Pad_Via, MountingHole:MountingHole_2.5mm_Pad_Via, F.Cu at (86.2, 85.0)
- moved VR1 132.8 mm to (96.3, 76.8), turned to 90 degrees
- moved U4 114.9 mm to (113.3, 82.8), turned to 90 degrees
- moved J2 104.3 mm to (86.5, 100.0)
- moved C5 100.1 mm to (87.0, 77.2), turned to -90 degrees
- moved U1 96.5 mm to (99.0, 100.5), turned to 180 degrees
- moved MK1 95.0 mm to (85.2, 62.3)
- moved LED1 94.8 mm to (82.3, 90.9), turned to 90 degrees
- moved FB1 94.4 mm to (103.5, 100.2), turned to 90 degrees
- moved C4 91.0 mm to (90.3, 77.3), turned to -90 degrees
- moved C2 90.9 mm to (96.5, 86.8), turned to 180 degrees
- moved R28 90.4 mm to (90.8, 62.8), turned to 180 degrees
- moved C6 90.3 mm to (99.0, 104.4)
- moved LED3 90.1 mm to (86.0, 91.0), turned to 90 degrees
- moved LED4 89.8 mm to (86.1, 72.0), turned to 180 degrees
- moved R9 89.6 mm to (82.3, 95.2), turned to -90 degrees
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Connections:
- MK1 pad OUT: Net-(U8-IN+) -> Net-(C17-Pad1)
- R28 pad 1: Net-(U8-IN+) -> Net-(C17-Pad1)
- R30 pad 1: GND -> Net-(C19-Pad2)
Other:
- board outline added: 89 x 55.5 mm

Commit message: regular
Parts:
- moved TP1 39.1 mm to (174.8, 65.8)
- moved TP2 39.1 mm to (174.8, 68.8)
- moved TP3 39.1 mm to (174.8, 71.9)
- moved TP4 39.1 mm to (174.8, 75.0)
- moved TP5 39.1 mm to (174.8, 78.0)
- moved REF** 2.28 mm to (115.7, 54.9)
- moved F1 1.00 mm to (106.8, 90.2)
- moved U4 0.59 mm to (112.8, 82.8)
- moved U5 0.54 mm to (113.2, 88.9)
- moved J4 0.50 mm to (107.0, 52.8)
Routing:
- net /ESP32-C3-02/SDA: track 0.00 -> 73.9 mm, vias 0 -> 4
- net /ESP32-C3-02/SCL: track 0.00 -> 71.1 mm, vias 0 -> 2
- net /VBAT: track 0.00 -> 10.7 mm
- net /USB_DN: track 0.00 -> 4.37 mm
- net /USB_DP: track 0.00 -> 4.37 mm
- net /ESP32-C3-02/USB_D-: track 0.00 -> 3.74 mm
- net /ESP32-C3-02/USB_D+: track 0.00 -> 3.74 mm
- net GND: vias 0 -> 4
- net /VBUS: vias 0 -> 3
- net /+5V_USB: vias 0 -> 3
- added copper zone on In1.Cu, net +3.3V
- added copper zone on F.Cu, net /+5V_USB
- added copper zone on In1.Cu, net /+5V_USB
- added copper zone on F.Cu, net /VBAT
- added copper zone on F.Cu, net /VBUS
- added copper zone on In1.Cu, net /VBUS
- added copper zone on F.Cu, net GND
- added copper zone on In2.Cu, net GND
