File: kicad_projects/260109-QCMD/main.kicad_sch (KiCad schematic)
At the start: 52 parts, among them U1 AD9851, U2 AD5252BRUZ1, U7 AD8007AKSZ-REEL7, U8 AD8310ARMZ, U9 LM7301IM5, Y1 ASE-30MHz

Commit message: regular
Parts:
- removed C42, C43, C44: 10n, symbol Device:C_Small
- removed C45, C47: 1u, symbol Device:C_Small
- removed C46: 100n, symbol Device:C_Small
- removed R24: 52R3, symbol Device:R
- removed R25, R26: 1k, symbol Device:R
- removed R27: 499, symbol Device:R
- removed U7: AD8007AKSZ-REEL7, KS_5_ADI, symbol AD8007AKSZ-REEL7:AD8007AKSZ-REEL7
- removed U8: AD8310ARMZ, RM_8_ADI, symbol AD8310ARMZ:AD8310ARMZ
- removed U9: LM7301IM5, LM7301IM5:SOT95P280X145-5N, symbol LM7301IM5:LM7301IM5
- added C10: 68p, symbol Device:C_Small
- added C12, C6: 47p, symbol Device:C_Small
- added C13: 100p, symbol Device:C_Small
- added C16: 15p, symbol Device:C_Small
- added C19, C9: 82p, symbol Device:C_Small
- added C50, C52: 1u, symbol Device:C_Small
- added C51: 100n, symbol Device:C_Small
- added J1, J2: Conn_Coaxial, symbol Connector:Conn_Coaxial
- added L5: 47n, symbol Device:L
- added L6: 72n, symbol Device:L
- added L7: 100n, symbol Device:L
- added R10: 0, symbol Device:R
- added R11, R12: 50, symbol Device:R
- added R28, R29: 10k, symbol Device:R
- added R30: 200, symbol Device:R
- added R32: 499, symbol Device:R
- added U12: AD8008ARZ-REEL7, R_8_ADI, symbol AD8008ARZ:AD8008ARZ-REEL7
- added U7: AD8302ARUZ-REEL, AD8302ARUZ-REEL:SOP65P640X120-14N, symbol AD8302ARUZ-REEL:AD8302ARUZ-REEL
- C29: value 3p9 -> 47p
- C30: value 1p -> 82p
- C31: value 18p -> 68p
- C32: value 2p4 -> 47p
- C33: value 2p7 -> 15p
- C34: value 18p -> 100p
- C35: value 2p2 -> 82p
- L2: value 510n -> 47n
- L3: value 750n -> 72n
- L4: value 390n -> 100n
- R15: value 100 -> 0
- R17, R18: value 200 -> 50
Connections:
- net +5V: no longer C22.1, C23.1, C24.1, C25.1, C26.1, C27.1, R14.1, U1.11 (AVDD), U1.18 (AVDD), U1.23 (DVDD), U1.6 (PVCC)
- net GND: now also U1.22 (RESET), C10.2, C13.2, C19.2, C51.2, C52.2, C6.2, J1.2 (Ext), J2.2 (Ext), R11.1, R12.1, R29.1, U12.4 (-VS); no longer R15.2
- net at R23.1: now also U12.6 (-IN2)
- net at R15.1: now also C16.1, C19.1, L7.2, R12.2; no longer U1.20 (IOUTB)
- net +5V_AD8007 renamed +5V_AD8008
- net +5V_AD8008: now also C51.1, C52.1, R28.2, U12.8 (+VS)
- net AD8007_IN+ renamed AD8008_IN1
- net AD8008_IN1: now also U12.3 (+IN1)
- net X_in: no longer names the net of R23.2
- net X_in: now also U12.7 (VOUT2)
- new net: J1.1 (In), R32.2, U12.1 (VOUT1)
- new net: C12.1, C13.1, C16.2, L6.2, L7.1
- new net: C50.1, R28.1, R29.2, R30.2
- new net: C50.2, R15.2
- new net: C10.1, C12.2, C9.1, L5.2, L6.1
- new net: C6.1, C9.2, L5.1, R10.2, R11.2
- new net: R10.1, U1.20 (IOUTB)
- new net: R32.1, U12.2 (-IN1)
- new net +5V_A: C22.1, C23.1, U1.11 (AVDD), U1.18 (AVDD)
- new net +5V_D: C24.1, C25.1, C26.1, C27.1, R14.1, U1.23 (DVDD), U1.6 (PVCC)
- new net AD8008_IN2: R30.1, U12.5 (+IN2)
- no-connect marks 9 -> 7
Other:
- sheet interface ports: added ADC0, ADC1; removed GAIN
- note added: "1kohm, 256 step"
- note added: "Iout = 39.93/RSET; RSET:(3,4)k --> Iout: (13.31,9.98)mA"
- note added: "input buffer"
- moved on the sheet: C20, C21, C37, C38, C39, C40, C41, R21, U2
