File: kicad_projects/260209-MSPM0-phil165/260209-MSPM0-phil165.kicad_pcb (KiCad board)
At the start: 2 copper layers, 53 x 28 mm, 37 parts, among them J1 USB4105-GF-A, J2 TC2030, U1 SPX3819M5-L-3-3, U2 CH340E, U3 MSPM0G3507SPTR, U4 LIS2DH, X1 8MHz

Commit message: regular
Parts:
- C10: value 1u -> 470n
- J1: value USB4105-GF-A -> USB4105-GF-A-060
- moved C3 1.77 mm to (62.8, 51.0)
- moved C4 1.77 mm to (66.0, 53.2)
- moved C5 1.77 mm to (69.2, 51.0)
- moved U1 1.77 mm to (66.0, 50.8)
- turned R2 to 180 degrees
Routing:
- net +3V3: track 10.4 -> 89.5 mm, vias 0 -> 8
- net +VBUS: track 0.00 -> 17.5 mm, vias 0 -> 2
- net +VBUSF: track 0.00 -> 15.0 mm
- net GND: track 0.00 -> 9.27 mm, vias 58 -> 117
- net /USBCC2: track 8.92 -> 5.74 mm
- net /UART0_RTS: track 29.0 -> 31.3 mm
- net /UART0_CTS: track 31.5 -> 33.7 mm
- net INT1: track 14.4 -> 16.6 mm
- net INT2: track 15.9 -> 17.9 mm
- net Net-(U1-BP): track 0.00 -> 1.70 mm
- added copper zone on F.Cu, net GND
Other:
- board text added: "MSPM0 Sensor, v0.1, 26/02/10, by hjin"
