File: kicad_projects/260209-MSPM0-phil165/260209-MSPM0-phil165.kicad_sch (KiCad schematic)
At the start: 0 parts

Commit message: regular
Parts:
- added C1: 10u, Capacitor_SMD:C_0805_2012Metric, symbol Device:C_Small
- added C2, C4, C7, C8: 470n, Capacitor_SMD:C_0805_2012Metric, symbol Device:C_Small
- added C3: 1u, Capacitor_SMD:C_0805_2012Metric, symbol Device:C_Small
- added C5, C6: 15p, Capacitor_SMD:C_0603_1608Metric, symbol Device:C_Small
- added J1: USB_C_Receptacle_USB2.0_16P, Connector_USB:USB_C_Receptacle_GCT_USB4105-xx-A_16P_TopMnt_Horizontal, symbol Connector:USB_C_Receptacle_USB2.0_16P
- added R1, R4: 0R, Resistor_SMD:R_0603_1608Metric, symbol Device:R_Small
- added R2: 5k1, Resistor_SMD:R_0603_1608Metric, symbol Device:R_Small
- added R3: 100k; 0.1%; 25ppm, Resistor_SMD:R_0603_1608Metric, symbol Device:R_Small
- added U1: MSPM0G3507SPTR, Package_QFP:LQFP-48_7x7mm_P0.5mm, symbol MSPM0G3507SPTR:MSPM0G3507SPTR
- added U2: USBLC6-2SC6, Package_TO_SOT_SMD:SOT-23-6, symbol Power_Protection:USBLC6-2SC6
- added U3: SPX3819M5-L-3-3, Package_TO_SOT_SMD:SOT-23-5, symbol Regulator_Linear:SPX3819M5-L-3-3
- added X1: 8MHz, Crystal:Crystal_SMD_3225-4Pin_3.2x2.5mm, symbol Device:Crystal_GND24_Small
Connections:
- new net: C8.1, R4.2
- new net: J1.A7 (D-), J1.B7 (D-), U2.1 (I/O1)
- new net: J1.A6 (D+), J1.B6 (D+), U2.3 (I/O2)
- new net: R3.2, U1.8 (PA2_ROSC)
- new net: J1.A1 (GND), J1.A12 (GND), J1.B1 (GND), J1.B12 (GND)
- new net +1V35: C2.1, U1.48 (VCORE)
- new net +3V3: C1.1, R2.1, U1.6 (VDD)
- new net +VBUS: C7.1, J1.A4 (VBUS), J1.A9 (VBUS), J1.B4 (VBUS), J1.B9 (VBUS), R4.1, U2.5 (VBUS)
- new net GND: C1.2, C2.2, C4.2, C5.2, C6.2, C7.2, C8.2, R1.2, R3.1, U1.7 (VSS), U2.2 (GND), X1.2 (G), X1.4 (G)
- new net HFXIN: C6.1, U1.11 (PA5_HFXIN), X1.1
- new net HFXOUT: C5.1, U1.12 (PA6_HFXOUT), X1.3
- new net NRST: C4.1, R2.2, U1.4 (RST_N)
- new net VREF+: C3.2, U1.43 (PA23_VREF+)
- new net VREF-: C3.1, R1.1, U1.39 (PA21_A1_7_VREF-)
Other:
- note added: "Guide of Xtal for MCU, refer to ST's AN2867"
- company: (none) -> hjin
- title: (none) -> MSPM0 Tutorial PCB

Commit message: regular
Parts:
- added C14, C4, C5, C6: 470n, Capacitor_SMD:C_0805_2012Metric, symbol Device:C_Small
- added C3, C7: 10u, Capacitor_SMD:C_0805_2012Metric, symbol Device:C_Small
- added J2: Conn_ARM_SWD_TagConnect_TC2030, Connector:Tag-Connect_TC2030-IDC-FP_2x03_P1.27mm_Vertical, symbol Connector:Conn_ARM_SWD_TagConnect_TC2030
- added R1, R3, R6, R7: 5k1, Resistor_SMD:R_0603_1608Metric, symbol Device:R_Small
- added U3: CH340E, Package_SO:MSOP-10_3x3mm_P0.5mm, symbol Interface_USB:CH340E
- added U5: LIS2DH, Package_LGA:LGA-14_2x2mm_P0.35mm_LayoutBorder3x4y, symbol Sensor_Motion:LIS2DH
- renumbered C7 to C1, C3 to C10, C1 to C11, C2 to C12, C4 to C13, C8 to C2, C6 to C8, C5 to C9, R4 to R2, R1 to R4, R3 to R5, R2 to R8, U2 to U1, U3 to U2, U1 to U4
Connections:
- net +3V3: now also U2.5 (OUT), C14.1, C7.1, J2.1 (VCC), R6.1, R7.1, U5.4 (~{CS}), U5.7 (Vdd_IO), U5.8 (Vdd)
- net GND: now also J1.A1 (GND), J1.A12 (GND), J1.B1 (GND), J1.B12 (GND), J1.S1 (SHIELD), U2.2 (GND), C14.2, C3.2, C4.2, C5.2, C6.2, C7.2, J2.5 (GND), R1.2, R3.2, U3.3 (GND), U5.10 (GND), U5.11 (GND), U5.12 (GND), U5.13 (GND), U5.14 (GND), U5.3 (SDO), U5.9 (GND)
- net NRST: now also J2.3 (~{RESET})
- net +VBUSF: now reaches C2.1, R2.2
- net +VBUSF: now also U2.1 (IN), U2.3 (EN), C3.1
- net USBCD-: now reaches J1.A7 (D-), J1.B7 (D-), U1.1 (I/O1)
- net USBCD+: now reaches J1.A6 (D+), J1.B6 (D+), U1.3 (I/O2)
- net USBD+: now reaches U1.4 (I/O2)
- net USBD+: now also U3.1 (UD+)
- net USBD-: now reaches U1.6 (I/O1)
- net USBD-: now also U3.2 (UD-)
- net UART0_TX: now reaches U4.1 (PA0)
- net UART0_TX: now also U3.9 (RXD)
- net I2C1_SCL: now reaches U4.14 (PB2)
- net I2C1_SCL: now also R7.2, U5.1 (SCL/SPC)
- net I2C1_SDA: now reaches U4.15 (PB3)
- net I2C1_SDA: now also R6.2, U5.2 (SDA/SDI)
- net UART0_RTS: now reaches U4.16 (PA8)
- net UART0_RTS: now also U3.5 (~{CTS})
- net UART0_CTS: now reaches U4.17 (PA9)
- net UART0_CTS: now also U3.4 (~{RTS})
- net UART0_RX: now reaches U4.2 (PA1)
- net UART0_RX: now also U3.8 (TXD)
- net INT1: now reaches U4.22 (PB8)
- net INT1: now also U5.6 (INT1)
- net INT2: now reaches U4.23 (PB9)
- net INT2: now also U5.5 (INT2)
- net SWDIO: now reaches U4.34 (PA19_SWDIO)
- net SWDIO: now also J2.2 (SWDIO)
- net SWCLK: now reaches U4.35 (PA20_SWCLK)
- net SWCLK: now also J2.4 (SWCLK)
- net USBCC1: now reaches J1.A5 (CC1)
- net USBCC1: now also R3.1
- net USBCC2: now reaches J1.B5 (CC2)
- net USBCC2: now also R1.1
- net at U2.4 (BP): now also C6.1
- new net: C4.1, C5.1, U3.10 (V3), U3.7 (VCC)
- no-connect marks 0 -> 32
Other:
- note added: "3.3V LDO"
- note added: "MCU"
- note added: "SWD"
- note added: "Sensor"
- note added: "USB to UART"
- moved on the sheet: C1, C10, C11, C12, C13, C2, C8, C9, J1, R2, R4, R5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

Commit message: regular
Parts:
- added FID1, FID2, FID3: Fiducial, Fiducial:Fiducial_1mm_Mask2mm, symbol Mechanical:Fiducial
- added H1, H2, H3, H4: M3, MountingHole:MountingHole_3.2mm_M3_Pad_Via, symbol Mechanical:MountingHole_Pad
- C1, C10, C11, C12, C2: footprint Capacitor_SMD:C_0805_2012Metric -> Capacitor_SMD:C_0603_1608Metric
- C13: renamed from C14; footprint Capacitor_SMD:C_0805_2012Metric -> Capacitor_SMD:C_0603_1608Metric
- C14: renamed from C13; footprint Capacitor_SMD:C_0805_2012Metric -> Capacitor_SMD:C_0603_1608Metric
- C4: renamed from C6; footprint Capacitor_SMD:C_0805_2012Metric -> Capacitor_SMD:C_0603_1608Metric
- C6: renamed from C4; footprint Capacitor_SMD:C_0805_2012Metric -> Capacitor_SMD:C_0603_1608Metric
- C7: renamed from C5; footprint Capacitor_SMD:C_0805_2012Metric -> Capacitor_SMD:C_0603_1608Metric
- J1: value USB_C_Receptacle_USB2.0_16P -> USB4105-GF-A
- J2: value Conn_ARM_SWD_TagConnect_TC2030 -> TC2030
- renumbered C7 to C5, U1 to D1, R2 to R1, R1 to R2, R5 to R4, R4 to R5, U2 to U1, U3 to U2, U4 to U3, U5 to U4
Connections:
- net +3V3: now also C6.1, C7.1, U2.10 (V3), U2.7 (VCC)
- net GND: now also H1.1, H2.1, H3.1, H4.1
- no-connect marks 32 -> 33
Other:
- moved on the sheet: C3, C4, C5, U1

Commit message: regular
Parts:
- C11: footprint Capacitor_SMD:C_0603_1608Metric -> Capacitor_SMD:C_0805_2012Metric
- renumbered C14 to C13, C13 to C14, R8 to R6, R6 to R7, R7 to R8
Connections:
- net I2C0_SDA: now reaches U3.18 (PA10)
- net I2C0_SDA: now also R7.2, U4.2 (SDA/SDI)
- net I2C0_SCL: now reaches U3.19 (PA11)
- net I2C0_SCL: now also R8.2, U4.1 (SCL/SPC)
- net ROSC: now reaches R4.2, U3.8 (PA2_ROSC)
- removed net I2C1_SCL: R8.2, U3.14 (PB2), U4.1 (SCL/SPC)
- removed net I2C1_SDA: R7.2, U3.15 (PB3), U4.2 (SDA/SDI)
Other:
- note added: "Accelerometer"
- note added: "from ACC"
- note added: "to MCU"
- note added: "to/from ACC"
- note added: "to/from MCU"
- note removed: "Sensor"
- moved on the sheet: C14, R7, R8, U4

Commit message: regular
Parts:
- C1, C12, C13, C14, C2: Digikey 1276-1039-2-ND -> 1276-2083-2-ND; LCSC C13967 -> C1623; MPN CL21B474KBFNNNE -> CL10B474KA8NNNC; Mouser 187-CL21B474KBFNNNE -> 187-CL10B474KA8NNNC
- C10: value 1u -> 470n; Digikey 1276-1029-2-ND -> 1276-2083-2-ND; LCSC C28323 -> C1623; MPN CL21B105KBFNNNE -> CL10B474KA8NNNC; Mouser 187-CL21B105KBFNNNE -> 187-CL10B474KA8NNNC
- C4, C6, C7: Digikey 1276-2891-2-ND -> 1276-2083-2-ND; LCSC C15850 -> C1623; MPN CL21A106KAYNNNE -> CL10B474KA8NNNC; Mouser 187-CL21A106KAYNNNE -> 187-CL10B474KA8NNNC
- C8, C9: Digikey (none) -> 1276-1296-2-ND; LCSC (none) -> C1644; MPN (none) -> CL10C150JB8NNNC; Manufacturer (none) -> Samsung Electro-Mechanics; Mouser (none) -> 187-CL10C150JB8NNNC
- D1: Digikey (none) -> 497-5235-2-ND; LCSC (none) -> C7519; MPN (none) -> USBLC6-2SC6; Manufacturer (none) -> STMicroelectronics; Mouser (none) -> 511-USBLC6-2SC6
- J1: value USB4105-GF-A -> USB4105-GF-A-060; Digikey 2073-USB4105-GF-ATR-ND -> CONN RCP USB2.0 TYP C 16P SMD RA; LCSC C3020560 -> C3025063; MPN USB4105-GF-A -> USB4105-GF-A-060; Mouser 640-USB4105-GF-A -> 640-USB4105-GF-A-060
- R1, R5: MFN YAGEO -> (none); MPN (none) -> RC0603FR-070RL; Manufacturer RC0603FR-070RL -> YAGEO
- R2, R3, R6, R7, R8: Digikey (none) -> 311-5.10KHRTR-ND; LCSC (none) -> C105580; MPN (none) -> RC0603FR-075K1L; Manufacturer (none) -> YAGEO; Mouser (none) -> 603-RC0603FR-075K1L
- R4: MFN RT0603BRD07100KL -> (none); MPN (none) -> RT0603BRD07100KL
- U1: value SPX3819M5-L-3-3 -> SPX3819M5-L-3-3/TR
- U2: LCSC (none) -> C99652; MPN (none) -> CH340E; Manufacturer (none) -> WCH
- U4: Digikey (none) -> 497-13795-2-ND; LCSC (none) -> C155670; MPN (none) -> LIS2DHTR; Manufacturer (none) -> STMicroelectronics; Mouser (none) -> 511-LIS2DHTR
Other:
- moved on the sheet: C5
